Commit message: hardware interface

File: description/ros2_control.xacro (robot description, xacro)
@@ -1,5 +1,5 @@
 <?xml version="1.0"?>
 <robot xmlns:xacro="http://www.ros.org/wiki/xacro">
-    <ros2_control name="GazeboSystem" type="system">
+    <!-- <ros2_control name="GazeboSystem" type="system">
         <hardware>
             <plugin>gazebo_ros2_control/GazeboSystem</plugin>
@@ -53,4 +53,48 @@
             <state_interface name="position"/>
         </joint>
+    </ros2_control> -->
+    <ros2_control name="ServoSystem" type="system">
+        <hardware>
+            <plugin>demo_arm/ServoBotSystemHardware</plugin>
+            <param name="rot_base_name">rot_base_joint</param>
+            <param name="arm1_name">arm1_joint</param>
+            <param name="arm2_name">arm2_joint</param>
+            <param name="arm3_name">arm3_joint</param>
+            <param name="claw_name">claw_joint</param>
+            <param name="loop_rate">30</param>
+            <param name="device">/dev/serial/by-path/platform-fd500000.pcie-pci-0000:01:00.0-usb-0:1.3:1.0-port0</param>
+            <param name="baud_rate">115200</param>
+            <param name="timeout">1000</param>
+        </hardware>
+        <joint name="rot_base_joint">
+            <command_interface name="velocity"/>
+            <state_interface name="velocity"/>
+            <state_interface name="position"/>
+        </joint>
+        <joint name="arm1_joint">
+            <command_interface name="velocity"/>
+            <state_interface name="velocity"/>
+            <state_interface name="position"/>
+        </joint>
+        <joint name="arm2_joint">
+            <command_interface name="velocity"/>
+            <state_interface name="velocity"/>
+            <state_interface name="position"/>
+        </joint>
+        <joint name="arm3_joint">
+           <command_interface name="velocity"/>
+            <state_interface name="velocity"/>
+            <state_interface name="position"/>
+        </joint>
+        <joint name="claw_joint">
+            <command_interface name="velocity"/>
+            <state_interface name="velocity"/>
+            <state_interface name="position"/>
+        </joint>
+        <!-- <joint name="right_claw_joint">
+            <command_interface name="velocity"/>
+            <state_interface name="velocity"/>
+            <state_interface name="position"/>
+        </joint> -->
     </ros2_control>
 </robot>
