Commit message: velocity controller configured

File: description/gazebo_control.xacro (robot description, xacro)
@@ -39,5 +39,5 @@
     <gazebo>
         <plugin name="gazebo_ros2_control" filename="libgazebo_ros2_control.so">
-            <parameters>$(find demo_arm)/config/joint_jog_control.yaml</parameters>
+            <parameters>$(find demo_arm)/config/vel_controller.yaml</parameters>
         </plugin>
     </gazebo>

File: description/inertial_macros.xacro (robot description, xacro)
@@ -24,6 +24,15 @@
             <mass value="${mass}" />
             <inertia ixx="${(2/5) * mass * (radius*radius)}" ixy="0.0" ixz="0.0"
-                    iyy="${(2/5) * mass * (radius*radius)}" iyz="0.0"
-                    izz="${(2/5) * mass * (radius*radius)}" />
+                     iyy="${(2/5) * mass * (radius*radius)}" iyz="0.0"
+                     izz="${(2/5) * mass * (radius*radius)}" />
+        </inertial>
+    </xacro:macro>
+    <xacro:macro name="inertial_bracket" params="mass length height width *origin">
+        <inertial>
+            <xacro:insert_block name="origin"/>
+            <mass value="${mass}"/>
+            <inertia ixx="${0.0}" ixy="0.0" ixz="0.0"
+                    iyy="${0.0}" iyz="0.0"
+                    izz="${0.0}" />
         </inertial>
     </xacro:macro>

File: description/robot.urdf.xacro (robot description, xacro)
@@ -2,4 +2,5 @@
 <robot xmlns:xacro="http://www.ros.org/wiki/xacro"  name="robot_arm">
     <xacro:include filename="robot_core.xacro"/>
-    <!-- <xacro:include filename="ros2_control.xacro"/> -->
+    <xacro:include filename="gazebo_control.xacro"/>
+    <xacro:include filename="ros2_control.xacro"/>
 </robot>

File: description/robot_core.xacro (robot description, xacro)
@@ -35,5 +35,5 @@
         </collision>
         <xacro:inertial_cylinder mass="0.5" radius="0.0475" length="0.045">
-            <origin xyz="0 0 0" rpy="0 0 0"/>
+            <origin xyz="0 0 0.0225" rpy="0 0 0"/>
         </xacro:inertial_cylinder>
     </link>
@@ -66,5 +66,5 @@
         </collision>
         <xacro:inertial_cylinder mass="0.2" radius="0.0475" length="0.01">
-            <origin xyz="0 0 0" rpy="0 0 0"/>
+            <origin xyz="0 0 0.005" rpy="0 0 0"/>
         </xacro:inertial_cylinder>
     </link>
@@ -88,6 +88,6 @@
             </geometry>
         </collision>
-        <xacro:inertial_box mass="0.5" x="0.04"  y="0.04" z="0.03">
-            <origin xyz="0 0 0" rpy="0 0 0"/>
+        <xacro:inertial_box mass="0.5" x="0.064"  y="0.04" z="0.03">
+            <origin xyz="0 0 0.015" rpy="0 0 0"/>
         </xacro:inertial_box>
     </link>
@@ -107,4 +107,7 @@
             </geometry>
         </collision>
+        <xacro:inertial_box mass="0.015" x="0.068"  y="0.025" z="0.087">
+            <origin xyz="-0.034 0 0.0745" rpy="${pi} 0 0"/>
+        </xacro:inertial_box>
     </link>
     <joint name="arm1_joint" type="revolute">
@@ -130,4 +133,7 @@
             </geometry>
         </collision>
+        <xacro:inertial_box mass="0.012" x="0.053"  y="0.025" z="0.057">
+            <origin xyz="0 0 0" rpy="0 0 0"/>
+        </xacro:inertial_box>
     </link>
     <joint name="arm_bracket_joint" type="fixed">
@@ -150,6 +156,6 @@
             </geometry>
         </collision>
-        <xacro:inertial_box mass="0.5" x="0.04"  y="0.04" z="0.03">
-            <origin xyz="0 0 0" rpy="0 0 0"/>
+        <xacro:inertial_box mass="0.5" x="0.049"  y="0.025" z="0.04">
+            <origin xyz="-0.026 0 -0.01" rpy="0 0 0"/>
         </xacro:inertial_box>
     </link>
@@ -175,4 +181,7 @@
             </geometry>
         </collision>
+        <xacro:inertial_cylinder mass="0.2" radius="0.006" length="0.07">
+            <origin xyz="0 0 0.035" rpy="0 0 0"/>
+        </xacro:inertial_cylinder>
     </link>
     <joint name="arm2_stem_joint" type="fixed">
@@ -196,6 +205,6 @@
             </geometry>
         </collision>
-        <xacro:inertial_box mass="0.5" x="0.04"  y="0.04" z="0.03">
-            <origin xyz="0 0 0" rpy="0 0 0"/>
+        <xacro:inertial_box mass="0.5" x="0.048"  y="0.025" z="0.04">
+            <origin xyz="0 0 0.02" rpy="0 0 0"/>
         </xacro:inertial_box>
     </link>
@@ -214,9 +223,12 @@
         </visual>
         <collision>
-            <origin xyz="-0.5 0.0125 0.0295" rpy="${pi} 0 0"/>
+            <origin xyz="-0.05 0.0125 0.0295" rpy="${pi} 0 0"/>
             <geometry>
                 <mesh filename="package://demo_arm/meshes/arm3_bracket.stl" scale="0.001 0.001 0.001"/>
             </geometry>
         </collision>
+        <xacro:inertial_box mass="0.008" x="0.053"  y="0.025" z="0.042">
+            <origin xyz="-0.025 0 0.0295" rpy="${pi} 0 0"/>
+        </xacro:inertial_box>
     </link>
     <joint name="arm3_joint" type="revolute">
@@ -237,11 +249,11 @@
         </visual>
         <collision>
-            <origin xyz="0 0 0"/>
+            <origin xyz="0 0 0.015"/>
             <geometry>
                 <box size="0.065 0.025 0.03"/>
             </geometry>
         </collision>
-        <xacro:inertial_box mass="0.5" x="0.04"  y="0.04" z="0.03">
-            <origin xyz="0 0 0" rpy="0 0 0"/>
+        <xacro:inertial_box mass="0.5" x="0.065"  y="0.025" z="0.03">
+            <origin xyz="0 0 0.015" rpy="0 0 0"/>
         </xacro:inertial_box>
     </link>
@@ -260,9 +272,12 @@
         </visual>
         <collision>
-            <origin xyz="0 0 0"/>
+            <origin xyz="0 0.01 0" rpy="${pi/2} 0 0"/>
             <geometry>
                 <mesh filename="package://demo_arm/meshes/right_claw.stl" scale="0.001 0.001 0.001"/>
             </geometry>
         </collision>
+        <xacro:inertial_box mass="0.008" x="0.015"  y="0.02" z="0.03">
+            <origin xyz="0.0075 0 0.015" rpy="${pi/2} 0 0"/>
+        </xacro:inertial_box>
     </link>
     <joint name="left_claw_joint" type="prismatic">
@@ -282,9 +297,12 @@
         </visual>
         <collision>
-            <origin xyz="0 0 0"/>
+            <origin xyz="-0.015 0.01 0" rpy="${pi/2} 0 0"/>
             <geometry>
                 <mesh filename="package://demo_arm/meshes/left_claw.stl" scale="0.001 0.001 0.001"/>
             </geometry>
         </collision>
+        <xacro:inertial_box mass="0.008" x="0.015"  y="0.02" z="0.03">
+            <origin xyz="-0.0075 0 0.015" rpy="${pi/2} 0 0"/>
+        </xacro:inertial_box>
     </link>
     <joint name="right_claw_joint" type="prismatic">

Commit message: CMakeList.txt modifications and nomenclature

File: description/gazebo_control.xacro (robot description, xacro)
@@ -42,3 +42,57 @@
         </plugin>
     </gazebo>
+    <!-- ___________________ Defining ros2_control parameters _______________________ -->
+    <ros2_control name="GazeboSystem" type="system">
+        <hardware>
+            <plugin>gazebo_ros2_control/GazeboSystem</plugin>
+        </hardware>
+        <joint name="rot_base_joint">
+            <command_interface name="velocity">
+                <param name="min">-10</param>
+                <param name="max">10</param>
+            </command_interface>
+            <state_interface name="velocity"/>
+            <state_interface name="position"/>
+        </joint>
+        <joint name="arm1_joint">
+            <command_interface name="velocity">
+                <param name="min">-10</param>
+                <param name="max">10</param>
+            </command_interface>
+            <state_interface name="velocity"/>
+            <state_interface name="position"/>
+        </joint>
+        <joint name="arm2_joint">
+            <command_interface name="velocity">
+                <param name="min">-10</param>
+                <param name="max">10</param>
+            </command_interface>
+            <state_interface name="velocity"/>
+            <state_interface name="position"/>
+        </joint>
+        <joint name="arm3_joint">
+            <command_interface name="velocity">
+                <param name="min">-10</param>
+                <param name="max">10</param>
+            </command_interface>
+            <state_interface name="velocity"/>
+            <state_interface name="position"/>
+        </joint>
+        <joint name="left_claw_joint">
+            <command_interface name="velocity">
+                <param name="min">-10</param>
+                <param name="max">10</param>
+            </command_interface>
+            <state_interface name="velocity"/>
+            <state_interface name="position"/>
+        </joint>
+        <joint name="right_claw_joint">
+            <command_interface name="velocity">
+                <param name="min">-10</param>
+                <param name="max">10</param>
+            </command_interface>
+            <state_interface name="velocity"/>
+            <state_interface name="position"/>
+        </joint>
+    </ros2_control>
 </robot>

File: description/robot.urdf.xacro (robot description, xacro)
@@ -3,7 +3,7 @@
     <!-- DEFINE robot properties : Links, Joints -->
     <xacro:include filename="robot_core.xacro"/>
-    <!-- Define the gazebo specific parameters -->
-    <xacro:include filename="gazebo_control.xacro"/>
-    <!-- Define ros2_control parameters -->
+    <!-- Define the gazebo specific parameters and gazebo_ros2_control plugin -->
+    <!-- <xacro:include filename="gazebo_control.xacro"/> -->
+    <!-- Define ros2_control parameters with hardware abstraction-->
     <xacro:include filename="ros2_control.xacro"/>
 </robot>

File: description/ros2_control.xacro (robot description, xacro)
@@ -1,60 +1,7 @@
 <?xml version="1.0"?>
 <robot xmlns:xacro="http://www.ros.org/wiki/xacro">
-    <!-- <ros2_control name="GazeboSystem" type="system">
-        <hardware>
-            <plugin>gazebo_ros2_control/GazeboSystem</plugin>
-        </hardware>
-        <joint name="rot_base_joint">
-            <command_interface name="velocity">
-                <param name="min">-10</param>
-                <param name="max">10</param>
-            </command_interface>
-            <state_interface name="velocity"/>
-            <state_interface name="position"/>
-        </joint>
-        <joint name="arm1_joint">
-            <command_interface name="velocity">
-                <param name="min">-10</param>
-                <param name="max">10</param>
-            </command_interface>
-            <state_interface name="velocity"/>
-            <state_interface name="position"/>
-        </joint>
-        <joint name="arm2_joint">
-            <command_interface name="velocity">
-                <param name="min">-10</param>
-                <param name="max">10</param>
-            </command_interface>
-            <state_interface name="velocity"/>
-            <state_interface name="position"/>
-        </joint>
-        <joint name="arm3_joint">
-            <command_interface name="velocity">
-                <param name="min">-10</param>
-                <param name="max">10</param>
-            </command_interface>
-            <state_interface name="velocity"/>
-            <state_interface name="position"/>
-        </joint>
-        <joint name="left_claw_joint">
-            <command_interface name="velocity">
-                <param name="min">-10</param>
-                <param name="max">10</param>
-            </command_interface>
-            <state_interface name="velocity"/>
-            <state_interface name="position"/>
-        </joint>
-        <joint name="right_claw_joint">
-            <command_interface name="velocity">
-                <param name="min">-10</param>
-                <param name="max">10</param>
-            </command_interface>
-            <state_interface name="velocity"/>
-            <state_interface name="position"/>
-        </joint>
-    </ros2_control> -->
     <ros2_control name="ServoSystem" type="system">
         <hardware>
-            <plugin>demo_arm/ServoBotSystemHardware</plugin>
+            <plugin>demo_arm/ServoSystemHardware</plugin>
             <param name="rot_base_name">rot_base_joint</param>
             <param name="arm1_name">arm1_joint</param>
