Commit message: urdf development

File: description/robot_core.xacro (robot description, xacro)
@@ -78,5 +78,5 @@
             <origin xyz="0 0 0.015"/>
             <geometry>
-                <box size="0.04 0.04 0.03"/>
+                <box size="0.064 0.04 0.03"/>
             </geometry>
             <material name="blue"/>
@@ -93,3 +93,41 @@
     </link>
     <!-- ____________________________ Arm1 ______________________ -->
+    <link name="arm1_bracket">
+        <visual>
+            <origin xyz="-0.068 0.0125 0.0745" rpy="${pi} 0 0"/>
+            <geometry>
+                <mesh filename="package://demo_arm/meshes/arm1_bracket.stl" scale="0.001 0.001 0.001"/>
+            </geometry>
+            <material name="orange"/>
+        </visual>
+        <collision>
+            <origin xyz="0 0 0"/>
+            <geometry>
+                <mesh filename="package://demo_arm/meshes/arm1_bracket.stl" scale="0.001 0.001 0.001"/>
+            </geometry>
+        </collision>
+    </link>
+    <joint name="arm1_joint" type="revolute">
+        <parent link="arm1_motor"/>
+        <child link="arm1_bracket"/>
+        <origin xyz="0.034 -0.014 0.022" rpy="0 0 0"/>
+        <axis xyz="1 0 0" rpy="0 0 0"/>
+        <limit lower="-${pi/2}" upper="${pi/2}" effort="100" velocity="0.2"/>
+    </joint>
+    <!-- ___________________________ Arm2 _______________________________ -->
+    <!-- <link name="arm2_bracket">
+        <visual>
+            <origin xyz="-0.034 0.0125 0.0745" rpy="${pi} 0 0"/>
+            <geometry>
+                <mesh filename="package://demo_arm/meshes/arm2_bracket.stl" scale="0.001 0.001 0.001"/>
+            </geometry>
+            <material name="orange"/>
+        </visual>
+        <collision>
+            <origin xyz="0 0 0"/>
+            <geometry>
+                <mesh filename="package://demo_arm/meshes/arm2_bracket.stl" scale="0.001 0.001 0.001"/>
+            </geometry>
+        </collision>
+    </link> -->
 </robot>

Commit message: urdf development

File: description/robot_core.xacro (robot description, xacro)
@@ -85,5 +85,5 @@
             <origin xyz="0 0 0.015"/>
             <geometry>
-                <box size="0.04 0.04 0.03"/>
+                <box size="0.064 0.04 0.03"/>
             </geometry>
         </collision>
@@ -99,8 +99,8 @@
                 <mesh filename="package://demo_arm/meshes/arm1_bracket.stl" scale="0.001 0.001 0.001"/>
             </geometry>
-            <material name="orange"/>
-        </visual>
-        <collision>
-            <origin xyz="0 0 0"/>
+            <material name="black"/>
+        </visual>
+        <collision>
+            <origin xyz="-0.068 0.0125 0.0745" rpy="${pi} 0 0"/>
             <geometry>
                 <mesh filename="package://demo_arm/meshes/arm1_bracket.stl" scale="0.001 0.001 0.001"/>
@@ -116,18 +116,114 @@
     </joint>
     <!-- ___________________________ Arm2 _______________________________ -->
-    <!-- <link name="arm2_bracket">
-        <visual>
-            <origin xyz="-0.034 0.0125 0.0745" rpy="${pi} 0 0"/>
+    <link name="arm2_bracket">
+        <visual>
+            <origin xyz="-0.0265 -0.0125 0"/>
             <geometry>
                 <mesh filename="package://demo_arm/meshes/arm2_bracket.stl" scale="0.001 0.001 0.001"/>
             </geometry>
-            <material name="orange"/>
-        </visual>
-        <collision>
+            <material name="black"/>
+        </visual>
+        <collision>
+            <origin xyz="-0.0265 -0.0125 0"/>
+            <geometry>
+                <mesh filename="package://demo_arm/meshes/arm2_bracket.stl" scale="0.001 0.001 0.001"/>
+            </geometry>
+        </collision>
+    </link>
+    <joint name="arm_bracket_joint" type="fixed">
+        <parent link="arm1_bracket"/>
+        <child link="arm2_bracket"/>
+        <origin xyz="-0.034 0 0.0745"/>
+    </joint>
+    <link name="arm2_motor">
+        <visual>
+            <origin xyz="-0.026 0 -0.01"/>
+            <geometry>
+                <box size="0.049 0.025 0.04"/>
+            </geometry>
+            <material name="blue"/>
+        </visual>
+        <collision>
+            <origin xyz="-0.026 0 -0.01"/>
+            <geometry>
+                <box size="0.049 0.025 0.04"/>
+            </geometry>
+        </collision>
+        <xacro:inertial_box mass="0.5" x="0.04"  y="0.04" z="0.03">
+            <origin xyz="0 0 0" rpy="0 0 0"/>
+        </xacro:inertial_box>
+    </link>
+    <joint name="arm2_joint" type="revolute">
+        <parent link="arm2_bracket"/>
+        <child link="arm2_motor"/>
+        <origin xyz="0.026 0 0.044"/>
+        <axis xyz="1 0 0" rpy="0 0 0"/>
+        <limit lower="-${pi/2}" upper="${pi/2}" effort="100" velocity="0.2"/>
+    </joint>
+    <link name="arm2_stem">
+        <visual>
             <origin xyz="0 0 0"/>
             <geometry>
-                <mesh filename="package://demo_arm/meshes/arm2_bracket.stl" scale="0.001 0.001 0.001"/>
-            </geometry>
-        </collision>
-    </link> -->
+                <mesh filename="package://demo_arm/meshes/arm2_stem.stl" scale="0.001 0.001 0.001"/>
+            </geometry>
+            <material name="white"/>
+        </visual>
+        <collision>
+            <origin xyz="0 0 0"/>
+            <geometry>
+                <mesh filename="package://demo_arm/meshes/arm2_stem.stl" scale="0.001 0.001 0.001"/>
+            </geometry>
+        </collision>
+    </link>
+    <joint name="arm2_stem_joint" type="fixed">
+        <parent link="arm2_motor"/>
+        <child link="arm2_stem"/>
+        <origin xyz="-0.0245 0 0.01"/>
+    </joint>
+    <!-- _____________________________ Arm3 ______________________________ -->
+    <link name="arm3_motor">
+        <visual>
+            <origin xyz="0 0 0.02"/>
+            <geometry>
+                <box size="0.048 0.025 0.04"/>
+            </geometry>
+            <material name="blue"/>
+        </visual>
+        <collision>
+            <origin xyz="0 0 0.02"/>
+            <geometry>
+                <box size="0.048 0.025 0.04"/>
+            </geometry>
+        </collision>
+        <xacro:inertial_box mass="0.5" x="0.04"  y="0.04" z="0.03">
+            <origin xyz="0 0 0" rpy="0 0 0"/>
+        </xacro:inertial_box>
+    </link>
+    <joint name="arm3_motor_joint" type="fixed">
+        <parent link="arm2_stem"/>
+        <child link="arm3_motor"/>
+        <origin xyz="0 0 0.07"/>
+    </joint>
+    <link name="arm3_bracket">
+        <visual>
+            <origin xyz="-0.05 0.0125 0.0415" rpy="${pi} 0 0"/>
+            <geometry>
+                <mesh filename="package://demo_arm/meshes/arm3_bracket.stl" scale="0.001 0.001 0.001"/>
+            </geometry>
+            <material name="black"/>
+        </visual>
+        <collision>
+            <origin xyz="-0.5 0.0125 0.0415" rpy="${pi} 0 0"/>
+            <geometry>
+                <mesh filename="package://demo_arm/meshes/arm3_bracket.stl" scale="0.001 0.001 0.001"/>
+            </geometry>
+        </collision>
+    </link>
+    <joint name="arm3_joint" type="revolute">
+        <parent link="arm3_motor"/>
+        <child link="arm3_bracket"/>
+        <origin xyz="0.024 0 0.035"/>
+        <axis xyz="1 0 0" rpy="0 0 0"/>
+        <limit lower="-${pi/2}" upper="${pi/2}" effort="100" velocity="0.2"/>
+    </joint>
 </robot>

Commit message: CMakeList.txt debugging

File: description/robot_core.xacro (robot description, xacro)
@@ -306,5 +306,5 @@
         </xacro:inertial_box>
     </link>
-    <joint name="right_claw_joint" type="prismatic">
+    <!-- <joint name="right_claw_joint" type="prismatic">
         <parent link="claw_base"/>
         <child link="right_claw"/>
@@ -312,4 +312,11 @@
         <axis xyz="1 0 0"/>
         <limit lower="-0.015" upper="0" effort="100" velocity="0.2"/>
+    </joint> -->
+    <joint name="right_claw_joint" type="prismatic">
+        <parent link="claw_base"/>
+        <child link="right_claw"/>
+        <origin xyz="0 0.0025 0.03" rpy="0 0 0"/>
+        <axis xyz="1 0 0"/>
+        <mimic joint="left_claw_joint" multiplier="1.0"/>
     </joint>
 </robot>

Commit message: fixed CMakeList.txt, organise launch files, create mimic right_claw_joint

File: description/robot_core.xacro (robot description, xacro)
@@ -318,5 +318,6 @@
         <origin xyz="0 0.0025 0.03" rpy="0 0 0"/>
         <axis xyz="1 0 0"/>
-        <mimic joint="left_claw_joint" multiplier="1.0"/>
+        <limit lower="-0.015" upper="0" effort="100" velocity="0.2"/>
+        <mimic joint="left_claw_joint" multiplier="-1.0"/>
     </joint>
 </robot>

File: description/ros2_control.xacro (robot description, xacro)
@@ -8,5 +8,5 @@
             <param name="arm2_name">arm2_joint</param>
             <param name="arm3_name">arm3_joint</param>
-            <param name="claw_name">claw_joint</param>
+            <param name="claw_name">left_claw_joint</param>
             <param name="loop_rate">30</param>
             <param name="device">/dev/serial/by-path/platform-fd500000.pcie-pci-0000:01:00.0-usb-0:1.3:1.0-port0</param>
@@ -34,14 +34,9 @@
             <state_interface name="position"/>
         </joint>
-        <joint name="claw_joint">
+        <joint name="left_claw_joint">
             <command_interface name="velocity"/>
             <state_interface name="velocity"/>
             <state_interface name="position"/>
         </joint>
-        <!-- <joint name="right_claw_joint">
-            <command_interface name="velocity"/>
-            <state_interface name="velocity"/>
-            <state_interface name="position"/>
-        </joint> -->
     </ros2_control>
 </robot>

Commit message: setting parameters for real-time

File: description/robot_core.xacro (robot description, xacro)
@@ -306,11 +306,4 @@
         </xacro:inertial_box>
     </link>
-    <!-- <joint name="right_claw_joint" type="prismatic">
-        <parent link="claw_base"/>
-        <child link="right_claw"/>
-        <origin xyz="0 0.0025 0.03"/>
-        <axis xyz="1 0 0"/>
-        <limit lower="-0.015" upper="0" effort="100" velocity="0.2"/>
-    </joint> -->
     <joint name="right_claw_joint" type="prismatic">
         <parent link="claw_base"/>

File: description/ros2_control.xacro (robot description, xacro)
@@ -10,5 +10,5 @@
             <param name="claw_name">left_claw_joint</param>
             <param name="loop_rate">30</param>
-            <param name="device">/dev/serial/by-path/platform-fd500000.pcie-pci-0000:01:00.0-usb-0:1.3:1.0-port0</param>
+            <param name="device">/dev/serial/by-id/usb-Silicon_Labs_CP2102_USB_to_UART_Bridge_Controller_0001-if00-port0</param>
             <param name="baud_rate">115200</param>
             <param name="timeout">1000</param>
