Commit message: control config and ros2_control

File: description/robot.urdf.xacro (robot description, xacro)
@@ -2,3 +2,4 @@
 <robot xmlns:xacro="http://www.ros.org/wiki/xacro"  name="robot_arm">
     <xacro:include filename="robot_core.xacro"/>
+    <!-- <xacro:include filename="ros2_control.xacro"/> -->
 </robot>

File: description/robot_core.xacro (robot description, xacro)
@@ -57,5 +57,5 @@
                 <cylinder radius="0.0475" length="0.01"/>
             </geometry>
-            <material name="white"/>
+            <material name="black"/>
         </visual>
         <collision>
@@ -111,5 +111,5 @@
         <parent link="arm1_motor"/>
         <child link="arm1_bracket"/>
-        <origin xyz="0.034 -0.014 0.022" rpy="0 0 0"/>
+        <origin xyz="0.034 -0.0075 0.022" rpy="0 0 0"/>
         <axis xyz="1 0 0" rpy="0 0 0"/>
         <limit lower="-${pi/2}" upper="${pi/2}" effort="100" velocity="0.2"/>
@@ -207,5 +207,5 @@
     <link name="arm3_bracket">
         <visual>
-            <origin xyz="-0.05 0.0125 0.0415" rpy="${pi} 0 0"/>
+            <origin xyz="-0.05 0.0125 0.0295" rpy="${pi} 0 0"/>
             <geometry>
                 <mesh filename="package://demo_arm/meshes/arm3_bracket.stl" scale="0.001 0.001 0.001"/>
@@ -214,5 +214,5 @@
         </visual>
         <collision>
-            <origin xyz="-0.5 0.0125 0.0415" rpy="${pi} 0 0"/>
+            <origin xyz="-0.5 0.0125 0.0295" rpy="${pi} 0 0"/>
             <geometry>
                 <mesh filename="package://demo_arm/meshes/arm3_bracket.stl" scale="0.001 0.001 0.001"/>
@@ -227,3 +227,71 @@
         <limit lower="-${pi/2}" upper="${pi/2}" effort="100" velocity="0.2"/>
     </joint>
+    <!-- ______________________________ Claw ___________________________________ -->
+    <link name="claw_base">
+        <visual>
+            <origin xyz="0 0 0.015"/>
+            <geometry>
+                <box size="0.065 0.025 0.03"/>
+            </geometry>
+            <material name="blue"/>
+        </visual>
+        <collision>
+            <origin xyz="0 0 0"/>
+            <geometry>
+                <box size="0.065 0.025 0.03"/>
+            </geometry>
+        </collision>
+        <xacro:inertial_box mass="0.5" x="0.04"  y="0.04" z="0.03">
+            <origin xyz="0 0 0" rpy="0 0 0"/>
+        </xacro:inertial_box>
+    </link>
+    <joint name="claw_base_joint" type="fixed">
+        <parent link="arm3_bracket"/>
+        <child link="claw_base"/>
+        <origin xyz="-0.024 0 0.0295"/>
+    </joint>
+    <link name="left_claw">
+        <visual>
+            <origin xyz="0 0.01 0" rpy="${pi/2} 0 0"/>
+            <geometry>
+                <mesh filename="package://demo_arm/meshes/right_claw.stl" scale="0.001 0.001 0.001"/>
+            </geometry>
+            <material name="black"/>
+        </visual>
+        <collision>
+            <origin xyz="0 0 0"/>
+            <geometry>
+                <mesh filename="package://demo_arm/meshes/right_claw.stl" scale="0.001 0.001 0.001"/>
+            </geometry>
+        </collision>
+    </link>
+    <joint name="left_claw_joint" type="prismatic">
+        <parent link="claw_base"/>
+        <child link="left_claw"/>
+        <origin xyz="0 0.0025 0.03"/>
+        <axis xyz="1 0 0"/>
+        <limit lower="0" upper="0.015" effort="100" velocity="0.2"/>
+    </joint>
+    <link name="right_claw">
+        <visual>
+            <origin xyz="-0.015 0.01 0" rpy="${pi/2} 0 0"/>
+            <geometry>
+                <mesh filename="package://demo_arm/meshes/left_claw.stl" scale="0.001 0.001 0.001"/>
+            </geometry>
+            <material name="black"/>
+        </visual>
+        <collision>
+            <origin xyz="0 0 0"/>
+            <geometry>
+                <mesh filename="package://demo_arm/meshes/left_claw.stl" scale="0.001 0.001 0.001"/>
+            </geometry>
+        </collision>
+    </link>
+    <joint name="right_claw_joint" type="prismatic">
+        <parent link="claw_base"/>
+        <child link="right_claw"/>
+        <origin xyz="0 0.0025 0.03"/>
+        <axis xyz="1 0 0"/>
+        <limit lower="-0.015" upper="0" effort="100" velocity="0.2"/>
+    </joint>
 </robot>
